Commit message: Black thrusters

File: urdf/ecn_auv.xacro (robot description, xacro)
@@ -12,5 +12,5 @@
 <xacro:property name="tl1" value=".1" />
 <xacro:property name="tr2" value=".05" />
-<xacro:property name="tl2" value=".05" />
+<xacro:property name="tl2" value=".03" />
 <xacro:property name="eps" value="0.00000001"/>
 <!-- Thruster link -->
@@ -20,4 +20,6 @@
         <child link="${name}"/>
         <origin rpy="${rpy}" xyz="${xyz}"/>
+        <dynamics damping="100.0" friction="100.0"/>
+        <limit effort="30" velocity="1.0" lower="-${eps}" upper="${eps}" />
     </joint>
     <link name="${name}">
@@ -29,7 +31,4 @@
                 <color rgba="0 0 0 1"/>
             </material>
-        <gazebo reference="${name}">
-            <material>Gazebo/Black</material>
-        </gazebo>
             </visual>
             <visual name="${name}_2">
@@ -41,9 +40,19 @@
                 <color rgba="0 0 0 1"/>
             </material>
-            <gazebo reference="${name}">
+            </visual>
+            <inertial>
+        <mass value="${eps}"/>
+        <inertia
+        ixx="${eps}"
+        ixy="0.0"
+        ixz="0.0"
+        iyy="${eps}"
+        iyz="0.0"
+        izz="${eps}"/>
+        </inertial>
+        </link>
+                <gazebo reference="${name}">
             <material>Gazebo/Black</material>
         </gazebo>
-            </visual>
-        </link>
 </xacro:macro>
 <!-- Plugin list -->

Commit message: added terrain

File: urdf/ecn_auv.xacro (robot description, xacro)
@@ -2,114 +2,114 @@
 <!-- STL-version of the URDF, used with gazebo for dynamic simulation  -->
 <robot name="ecn_auv" xmlns:xacro="http://www.ros.org/wiki/xacro">
-<xacro:property name="PI" value="3.1415926535897931"/>
-<!-- Body properties -->
-<xacro:property name="body_mass" value="25"/>
-<xacro:property name="body_radius" value="0.13"/>
-<xacro:property name="body_length" value="1.5" />
-<xacro:property name="X_cob" value="${body_radius*2}" />
-<!-- thrusters -->
-<xacro:property name="tr1" value=".02" />
-<xacro:property name="tl1" value=".1" />
-<xacro:property name="tr2" value=".05" />
-<xacro:property name="tl2" value=".03" />
-<xacro:property name="eps" value="0.00000001"/>
-<!-- Thruster link -->
-<xacro:macro name="thruster_link" params="name xyz rpy">
-    <joint name="${name}" type="fixed">
-        <parent link="base_link"/>
-        <child link="${name}"/>
-        <origin rpy="${rpy}" xyz="${xyz}"/>
-        <dynamics damping="100.0" friction="100.0"/>
-        <limit effort="30" velocity="1.0" lower="-${eps}" upper="${eps}" />
-    </joint>
-    <link name="${name}">
+    <xacro:property name="PI" value="3.1415926535897931"/>
+    <!-- Body properties -->
+    <xacro:property name="body_mass" value="25"/>
+    <xacro:property name="body_radius" value="0.13"/>
+    <xacro:property name="body_length" value="1.5" />
+    <xacro:property name="X_cob" value="${body_radius*2}" />
+    <!-- thrusters -->
+    <xacro:property name="tr1" value=".02" />
+    <xacro:property name="tl1" value=".1" />
+    <xacro:property name="tr2" value=".05" />
+    <xacro:property name="tl2" value=".03" />
+    <xacro:property name="eps" value="0.00000001"/>
+    <!-- Thruster link -->
+    <xacro:macro name="thruster_link" params="name xyz rpy">
+        <joint name="${name}" type="fixed">
+            <parent link="base_link"/>
+            <child link="${name}"/>
+            <origin rpy="${rpy}" xyz="${xyz}"/>
+            <dynamics damping="100.0" friction="100.0"/>
+            <limit effort="30" velocity="1.0" lower="-${eps}" upper="${eps}" />
+        </joint>
+        <link name="${name}">
             <visual name="${name}_1">
-            <geometry>
-                <cylinder length="${tl1}" radius="${tr1}"/>
-            </geometry>
-            <material name="black">
-                <color rgba="0 0 0 1"/>
-            </material>
+                <geometry>
+                    <cylinder length="${tl1}" radius="${tr1}"/>
+                </geometry>
+                <material name="black">
+                    <color rgba="0 0 0 1"/>
+                </material>
             </visual>
             <visual name="${name}_2">
-            <origin xyz="0 0 -${(tl1+tl2)/2}"/>
-            <geometry>
-                <cylinder length="${tl2}" radius="${tr2}"/>
-            </geometry>
-            <material name="black">
-                <color rgba="0 0 0 1"/>
-            </material>
+                <origin xyz="0 0 -${(tl1+tl2)/2}"/>
+                <geometry>
+                    <cylinder length="${tl2}" radius="${tr2}"/>
+                </geometry>
+                <material name="black">
+                    <color rgba="0 0 0 1"/>
+                </material>
             </visual>
             <inertial>
-        <mass value="${eps}"/>
-        <inertia
-        ixx="${eps}"
-        ixy="0.0"
-        ixz="0.0"
-        iyy="${eps}"
-        iyz="0.0"
-        izz="${eps}"/>
-        </inertial>
-        </link>
-                <gazebo reference="${name}">
-            <material>Gazebo/Black</material>
+                <mass value="${eps}"/>
+                <inertia
+                    ixx="${eps}"
+                    ixy="0.0"
+                    ixz="0.0"
+                    iyy="${eps}"
+                    iyz="0.0"
+                    izz="${eps}"/>
+                </inertial>
+            </link>
+            <gazebo reference="${name}">
+                <material>Gazebo/Black</material>
+            </gazebo>
+        </xacro:macro>
+        <!-- Plugin list -->
+        <gazebo>
+            <!-- Gazebo plugin listens to the body-->
+            <plugin name="freefloating_gazebo_control" filename="libfreefloating_gazebo_control.so">
+                <switchService>switch</switchService>
+                <updateRate>100</updateRate>
+                <link>base_link</link>
+                <!-- for each thruster, give the map to XYZ+RPY and the maximum effort -->
+                <thruster>
+                    <map>-1 0 0 0 0 ${-body_radius}</map>
+                    <effort>30</effort>
+                </thruster>
+                <thruster>
+                    <map>-1 0 0 0 0 ${body_radius}</map>
+                    <effort>30</effort>
+                </thruster>
+                <thruster>
+                    <map>0 1 0 0 0 0</map>
+                    <effort>30</effort>
+                </thruster>
+                <thruster>
+                    <map>0 0 -1 0 0 0</map>
+                    <effort>30</effort>
+                </thruster>
+                <thruster>
+                    <map>0 0 -1 0 ${2*X_cob} 0</map>
+                    <effort>30</effort>
+                </thruster>
+            </plugin>
         </gazebo>
-</xacro:macro>
-<!-- Plugin list -->
-    <gazebo>
-    <!-- Gazebo plugin listens to the body-->
-    <plugin name="freefloating_gazebo_control" filename="libfreefloating_gazebo_control.so">
-        <switchService>switch</switchService>
-        <updateRate>100</updateRate>
-        <link>base_link</link>
-        <!-- for each thruster, give the map to XYZ+RPY and the maximum effort -->
-        <thruster>
-            <map>-1 0 0 0 0 ${-body_radius}</map>
-            <effort>30</effort>
-        </thruster>
-        <thruster>
-            <map>-1 0 0 0 0 ${body_radius}</map>
-            <effort>30</effort>
-        </thruster>
-        <thruster>
-            <map>0 1 0 0 0 0</map>
-            <effort>30</effort>
-        </thruster>
-        <thruster>
-            <map>0 0 -1 0 0 0</map>
-            <effort>30</effort>
-        </thruster>
-        <thruster>
-            <map>0 0 -1 0 ${2*X_cob} 0</map>
-            <effort>30</effort>
-        </thruster>
-    </plugin>
-    </gazebo>
-<link name="base_link">
-    <visual>
-    <origin rpy="0 ${-PI/2} 0"/>
-    <geometry>
-        <cylinder length="${body_length}" radius="${body_radius}"/>
-    </geometry>
-    </visual>
-    <inertial>
-        <origin xyz="0 0 -${X_cob}" rpy="0 ${-PI/2} 0"/>
-        <mass value="${body_mass}"/>
-        <inertia
-        ixx="${body_mass*(body_radius*body_radius/4+body_length*body_length/12)}"
-        ixy="0.0"
-        ixz="0.0"
-        iyy="${body_mass*(body_radius*body_radius/4+body_length*body_length/12)}"
-        iyz="0.0"
-        izz="${body_mass*body_radius*body_radius/2}"/>
-        </inertial>
-<buoyancy>
-    <compensation>1.01</compensation>
-    <origin xyz= "0 0 ${X_cob}"/>
-    <limit radius="${body_radius}"/>
-    <damping xyz="60 100 100" rpy="20 50 50"/>
-</buoyancy>
-</link>
-    <xacro:thruster_link name="fwd_left" xyz="${-body_length/3} ${body_radius+tr2} 0" rpy="0 ${PI/2} 0"/>
-    <xacro:thruster_link name="fwd_right" xyz="${-body_length/3} -${body_radius+tr2} 0" rpy="0 ${PI/2} 0"/>
-</robot>
+        <link name="base_link">
+            <visual>
+                <origin rpy="0 ${-PI/2} 0"/>
+                <geometry>
+                    <cylinder length="${body_length}" radius="${body_radius}"/>
+                </geometry>
+            </visual>
+            <inertial>
+                <origin xyz="0 0 -${X_cob}" rpy="0 ${-PI/2} 0"/>
+                <mass value="${body_mass}"/>
+                <inertia
+                    ixx="${body_mass*(body_radius*body_radius/4+body_length*body_length/12)}"
+                    ixy="0.0"
+                    ixz="0.0"
+                    iyy="${body_mass*(body_radius*body_radius/4+body_length*body_length/12)}"
+                    iyz="0.0"
+                    izz="${body_mass*body_radius*body_radius/2}"/>
+                </inertial>
+                <buoyancy>
+                    <compensation>1.01</compensation>
+                    <origin xyz= "0 0 ${X_cob}"/>
+                    <limit radius="${body_radius}"/>
+                    <damping xyz="60 100 100" rpy="20 50 50"/>
+                </buoyancy>
+            </link>
+            <xacro:thruster_link name="fwd_left" xyz="${-body_length/3} ${body_radius+tr2} 0" rpy="0 ${PI/2} 0"/>
+            <xacro:thruster_link name="fwd_right" xyz="${-body_length/3} -${body_radius+tr2} 0" rpy="0 ${PI/2} 0"/>
+        </robot>

Commit message: Updates position sp topic & type

File: urdf/ecn_auv.xacro (robot description, xacro)
@@ -7,5 +7,5 @@
     <xacro:property name="body_radius" value="0.13"/>
     <xacro:property name="body_length" value="1.5" />
-    <xacro:property name="X_cob" value="${body_radius*2}" />
+    <xacro:property name="X_cog" value="${-0.5*body_radius}" />
     <!-- thrusters -->
     <xacro:property name="tr1" value=".02" />
@@ -20,8 +20,10 @@
             <child link="${name}"/>
             <origin rpy="${rpy}" xyz="${xyz}"/>
-            <dynamics damping="100.0" friction="100.0"/>
-            <limit effort="30" velocity="1.0" lower="-${eps}" upper="${eps}" />
+            <dynamics damping="10.0"/>
+            <axis xyz="0 1 0"/>
+            <limit effort="30" velocity="5.0" lower="-${PI/2}" upper="${PI/2}" />
         </joint>
         <link name="${name}">
+            <buoyancy><compensation>1.0</compensation></buoyancy>
             <visual name="${name}_1">
                 <geometry>
@@ -42,12 +44,12 @@
             </visual>
             <inertial>
-                <mass value="${eps}"/>
+                <mass value=".1"/>
                 <inertia
-                    ixx="${eps}"
+                    ixx=".1"
                     ixy="0.0"
                     ixz="0.0"
-                    iyy="${eps}"
+                    iyy=".1"
                     iyz="0.0"
-                    izz="${eps}"/>
+                    izz=".1"/>
                 </inertial>
             </link>
@@ -65,9 +67,9 @@
                 <!-- for each thruster, give the map to XYZ+RPY and the maximum effort -->
                 <thruster>
-                    <map>-1 0 0 0 0 ${-body_radius}</map>
+                    <map>-1 0 0 0 0 ${body_length/3}</map>
                     <effort>30</effort>
                 </thruster>
                 <thruster>
-                    <map>-1 0 0 0 0 ${body_radius}</map>
+                    <map>-1 0 0 0 0 ${-body_length/3}</map>
                     <effort>30</effort>
                 </thruster>
@@ -77,9 +79,9 @@
                 </thruster>
                 <thruster>
-                    <map>0 0 -1 0 0 0</map>
+                    <map>0 0 -1 0 ${-0.3*body_length} 0</map>
                     <effort>30</effort>
                 </thruster>
                 <thruster>
-                    <map>0 0 -1 0 ${2*X_cob} 0</map>
+                    <map>0 0 -1 0 ${0.3*body_length} 0</map>
                     <effort>30</effort>
                 </thruster>
@@ -94,5 +96,5 @@
             </visual>
             <inertial>
-                <origin xyz="0 0 -${X_cob}" rpy="0 ${-PI/2} 0"/>
+                <origin xyz="0 0 ${X_cog}" rpy="0 ${-PI/2} 0"/>
                 <mass value="${body_mass}"/>
                 <inertia
@@ -106,10 +108,9 @@
                 <buoyancy>
                     <compensation>1.01</compensation>
-                    <origin xyz= "0 0 ${X_cob}"/>
+                    <origin xyz= "0 0 0"/>
                     <limit radius="${body_radius}"/>
                     <damping xyz="60 100 100" rpy="20 50 50"/>
                 </buoyancy>
-            </link>
-            <gazebo>
+   <gazebo>
     <plugin name="imu_plugin" filename="libgazebo_ros_imu.so">
         <alwaysOn>true</alwaysOn>
@@ -121,5 +122,6 @@
     </plugin>
 </gazebo>
-            <xacro:thruster_link name="fwd_left" xyz="${-body_length/3} ${body_radius+tr2} 0" rpy="0 ${PI/2} 0"/>
-            <xacro:thruster_link name="fwd_right" xyz="${-body_length/3} -${body_radius+tr2} 0" rpy="0 ${PI/2} 0"/>
+            </link>
+    <xacro:thruster_link name="fwd_left" xyz="${-body_length/3} ${body_radius+tr2} 0" rpy="0 ${PI/2} 0"/>
+    <xacro:thruster_link name="fwd_right" xyz="${-body_length/3} -${body_radius+tr2} 0" rpy="0 ${PI/2} 0"/>
         </robot>
