Commit message: collision

File: urdf/auv.xacro (robot description, xacro)
@@ -95,4 +95,10 @@
                 </geometry>
             </visual>
+            <collision>
+                <origin rpy="0 ${-PI/2} 0"/>
+                <geometry>
+                    <cylinder length="${body_length}" radius="${body_radius}"/>
+                </geometry>
+            </collision>
             <inertial>
                 <origin xyz="0 0 ${X_cog}" rpy="0 ${-PI/2} 0"/>
