Commit message: with Blurr robot

File: urdf/brov2.xacro (robot description, xacro)
@@ -44,5 +44,5 @@
       <origin rpy="1.57079632679 0 1.57079632679" xyz="0.1 -0.167 -0.19"/>
       <geometry>
-        <mesh filename="file:///home/olivier/code/ros/src/ecn/rasom/ecn_rasom/ecn_rasom/urdf/brov2.stl" scale="0.001 0.001 0.001"/>
+        <mesh filename="package://ecn_rasom/urdf/brov2.stl" scale="0.001 0.001 0.001"/>
       </geometry>
     </visual>

Commit message: add bluerob2 mesh

File: urdf/brov2.xacro (robot description, xacro)
@@ -5,4 +5,7 @@
 <!-- =================================================================================== -->
 <robot name="auv">
+        <material name="brovgrey">
+    <color rgba="0.25 0.25 0.3 1"/>
+  </material>
   <!-- Plugin list -->
   <gazebo>
@@ -46,4 +49,5 @@
         <mesh filename="package://ecn_rasom/urdf/brov2.stl" scale="0.001 0.001 0.001"/>
       </geometry>
+      <material name="brovgrey"/>
     </visual>
     <inertial>

Commit message: gazebo color

File: urdf/brov2.xacro (robot description, xacro)
@@ -4,8 +4,9 @@
 <!-- |    EDITING THIS FILE BY HAND IS NOT RECOMMENDED                                 | -->
 <!-- =================================================================================== -->
-<robot name="auv">
-        <material name="brovgrey">
-    <color rgba="0.25 0.25 0.3 1"/>
-  </material>
+<robot name="auv" xmlns:xacro="http://www.ros.org/wiki/xacro">
+<xacro:property name="body_RGB" value="0.25 0.25 0.28"/>
+<material name="brovgrey">
+<color rgba="${body_RGB} 1"/>
+</material>
   <!-- Plugin list -->
   <gazebo>
@@ -43,4 +44,14 @@
     </plugin>
   </gazebo>
+  <gazebo reference="base_link">
+    <visual>
+    <material>
+      <ambient>${body_RGB} 1.0</ambient>
+      <diffuse>${body_RGB} 1.0</diffuse>
+      <specular>${body_RGB} 1.0</specular>
+      <emissive>0.0 0.0 0.0 0.0</emissive>
+    </material>
+  </visual>
+ </gazebo>
   <link name="base_link">
     <visual>

Commit message: better ekf

File: urdf/brov2.xacro (robot description, xacro)
@@ -148,9 +148,4 @@
     <origin rpy="0 0 -1.57079632679" xyz=".12 0.018 0.02"/>
 </joint>
-<joint name="mpu" type="fixed">
-    <parent link="base_link"/>
-    <child link="mpu"/>
-    <origin rpy="0 0 -1.57079632679" xyz=".13 0.018 0.02"/>
-</joint>
     <gazebo reference="lsm">
     <sensor name="imu_sensor" type="imu">
@@ -163,10 +158,15 @@
         <updateRateHZ>1000.0</updateRateHZ>
         <gaussianNoise>0.001</gaussianNoise>
-        <xyzOffset>0 0 0</xyzOffset>
-        <rpyOffset>0 0 0</rpyOffset>
+        <xyzOffset>.12 0.018 0.02</xyzOffset>
+        <rpyOffset>0 0 -1.57079632679</rpyOffset>
         <frameName>lsm</frameName>
     </plugin>
     </sensor>
 </gazebo>
+<joint name="mpu" type="fixed">
+    <parent link="base_link"/>
+    <child link="mpu"/>
+    <origin rpy="0 0 -1.57079632679" xyz=".13 0.018 0.02"/>
+</joint>
     <gazebo reference="mpu">
     <sensor name="imu_sensor" type="imu">
@@ -179,6 +179,6 @@
         <updateRateHZ>1000.0</updateRateHZ>
         <gaussianNoise>0.001</gaussianNoise>
-        <xyzOffset>0 0 0</xyzOffset>
-        <rpyOffset>0 0 0</rpyOffset>
+        <xyzOffset>.13 0.018 0.02</xyzOffset>
+        <rpyOffset>0 0 -1.57079632679</rpyOffset>
         <frameName>mpu</frameName>
     </plugin>

Commit message: imu alignment

File: urdf/brov2.xacro (robot description, xacro)
@@ -146,5 +146,5 @@
     <parent link="base_link"/>
     <child link="lsm"/>
-    <origin rpy="0 0 -1.57079632679" xyz=".12 0.018 0.02"/>
+    <origin rpy="0 0 0" xyz=".12 0.018 0.02"/>
 </joint>
     <gazebo reference="lsm">
@@ -159,5 +159,5 @@
         <gaussianNoise>0.001</gaussianNoise>
         <xyzOffset>.12 0.018 0.02</xyzOffset>
-        <rpyOffset>0 0 -1.57079632679</rpyOffset>
+        <rpyOffset>0 0 0</rpyOffset>
         <frameName>lsm</frameName>
     </plugin>
@@ -167,5 +167,5 @@
     <parent link="base_link"/>
     <child link="mpu"/>
-    <origin rpy="0 0 -1.57079632679" xyz=".13 0.018 0.02"/>
+    <origin rpy="0 0 0" xyz=".13 0.018 0.02"/>
 </joint>
     <gazebo reference="mpu">
@@ -180,5 +180,5 @@
         <gaussianNoise>0.001</gaussianNoise>
         <xyzOffset>.13 0.018 0.02</xyzOffset>
-        <rpyOffset>0 0 -1.57079632679</rpyOffset>
+        <rpyOffset>0 0 0</rpyOffset>
         <frameName>mpu</frameName>
     </plugin>
