Commit message: Noetic

File: urdf/brov2.urdf (robot description, URDF)
Before this commit: robot brov, 8 links, 7 joints
Links:
- link base_link: geometry visual mesh filename=urdf/brov2.ive scale=0.001 0.001 0.001

Commit message: dae mesh

File: urdf/brov2.urdf (robot description, URDF)
Before this commit: robot brov, 8 links, 7 joints
Links:
- added link lsm
- added link mpu
- link base_link: geometry visual mesh filename=package://ecn_rasom/urdf/bluerov2_noprop.dae
Joints:
- added joint lsm: type fixed, parent base_link, child lsm, origin xyz=.12 0.018 0.02 rpy=0 0 0
- added joint mpu: type fixed, parent base_link, child mpu, origin xyz=.13 0.018 0.02 rpy=0 0 0

File: urdf/brov2.xacro (robot description, xacro)
@@ -56,7 +56,6 @@
   <link name="base_link">
     <visual>
-      <origin rpy="1.57079632679 0 1.57079632679" xyz="0.1 -0.167 -0.19"/>
       <geometry>
-        <mesh filename="package://ecn_rasom/urdf/brov2.stl" scale="0.001 0.001 0.001"/>
+        <mesh filename="package://ecn_rasom/urdf/bluerov2_noprop.dae"/>
       </geometry>
       <material name="brovgrey"/>

Commit message: higher gains

File: urdf/brov2.urdf (robot description, URDF)
Before this commit: robot auv, 10 links, 9 joints
Links:
- link base_link: geometry visual mesh filename=bluerov2_noprop.dae
